Commit message: Implement Gazebo ROS 2 Nav2 RViz synchronization

File: src/openamrobot_description/urdf/gazebo_control.xacro (robot description, xacro)
@@ -153,4 +153,13 @@
     </sensor>
   </gazebo>
+  <!-- ── Link-level: imu_link ────────────────────────────────────── -->
+  <gazebo reference="imu_link">
+    <sensor name="imu_sensor" type="imu">
+      <topic>/imu</topic>
+      <update_rate>100</update_rate>
+      <always_on>true</always_on>
+      <visualize>false</visualize>
+    </sensor>
+  </gazebo>
   <!-- ── Link-level: lidar_link — sensor ONLY here ─────────────────── -->
   <gazebo reference="lidar_link">

File: src/openamrobot_description/urdf/robo_urdf.urdf.xacro (robot description, xacro)
@@ -621,5 +621,5 @@
     type="fixed">
     <origin
-      xyz="0.0 0.0 0.30"
+      xyz="0.35135 -0.0010251 0.1683"
       rpy="0 0 0" />
     <parent
@@ -664,4 +664,18 @@
     <child link="camera_optical_frame"/>
   </joint>
+  <!-- IMU frame kept separate from base_link so recorded data and hardware
+       deployments can preserve the physical sensor frame contract. -->
+  <link name="imu_link">
+    <inertial>
+      <mass value="0.01"/>
+      <inertia ixx="0.000001" ixy="0" ixz="0"
+               iyy="0.000001" iyz="0" izz="0.000001"/>
+    </inertial>
+  </link>
+  <joint name="imu_joint" type="fixed">
+    <origin xyz="0 0 0.12" rpy="0 0 0"/>
+    <parent link="base_link"/>
+    <child link="imu_link"/>
+  </joint>
   <xacro:include filename="gazebo_control.xacro" />
 </robot>
